Commit message: Initial changes

File: simulation/robots/go1_description/xacro/robot.xacro (robot description, xacro)
@@ -6,6 +6,16 @@
     <!-- <xacro:include filename="$(find go1_description)/xacro/stairs.xacro"/> -->
     <xacro:include filename="$(find go1_description)/xacro/gazebo.xacro"/>
-    <xacro:include filename="$(find go1_description)/xacro/depthCamera.xacro"/>
-    <xacro:include filename="$(find go1_description)/xacro/ultraSound.xacro"/>
+    <!-- <xacro:include filename="$(find go1_description)/xacro/depthCamera.xacro"/> -->
+    <!-- <xacro:include filename="$(find go1_description)/xacro/ultraSound.xacro"/> -->
+    <!-- <xacro:include filename="$(find go1_gazebo)/launch/stairs.urdf.xacro"/> -->
+    <xacro:if value="$(arg USE_CAMERA)">
+        <xacro:include filename="$(find a1_description)/xacro/realsense_d435.xacro"/>
+    </xacro:if>
+    <xacro:if value="$(arg USE_LIDAR)">
+        <xacro:include filename="$(find go1_description)/xacro/VLP-16.xacro"/>
+    </xacro:if>
+    <xacro:if value="$(arg USE_GPS)">
+        <xacro:include filename="$(find go1_description)/xacro/gps_gazebo.xacro"/>
+    </xacro:if>
     <!-- <xacro:include filename="$(find go1_gazebo)/launch/stairs.urdf.xacro"/> -->
     <!-- <xacro:stairs stairs="15" xpos="0" ypos="0" zpos="0" /> -->
@@ -57,4 +67,14 @@
         </inertial>
     </link>
+    <xacro:if value="$(arg USE_CAMERA)">
+        <xacro:realsense_d435 sensor_name="d435" parent_link="trunk" rate="10">
+            <origin rpy="0 0 0 " xyz="0.25 0 0.055"/>
+        </xacro:realsense_d435>
+    </xacro:if>
+    <xacro:if value="$(arg USE_LIDAR)">
+        <xacro:VLP-16 sensor_name="velodyne" parent= "trunk" rate= "10">
+            <origin rpy="0 0 0 " xyz="0 0 0.055"/>
+        </xacro:VLP-16>
+    </xacro:if>
     <xacro:if value="${(rolloverProtection == 'true')}">
         <joint name="stick_joint" type="fixed">
@@ -69,5 +89,5 @@
                 </geometry>
                 <origin rpy="0 0 0" xyz="0 0 0"/>
-                <!-- <material name="white"/> -->
+                <material name="white"/>
             </visual>
             <collision>
@@ -102,5 +122,5 @@
                 <box size="0.001 0.001 0.001"/>
             </geometry>
-            <!-- <material name="red"/> -->
+            <material name="red"/>
         </visual>
         <collision>
@@ -123,5 +143,5 @@
         <origin rpy="0 0 0" xyz="${-leg_offset_x} ${leg_offset_y} 0"/>
     </xacro:leg>
-    <xacro:depthCamera camID="1" name="face">
+    <!-- <xacro:depthCamera camID="1" name="face">
         <origin rpy="${PI} 0 0" xyz="0.2785 0.0125 0.0167"/>
     </xacro:depthCamera>
@@ -160,4 +180,4 @@
     <xacro:ultraSound name="face">
         <origin rpy="0 0 0" xyz="0.2747 0.0 -0.0088"/>
-    </xacro:ultraSound>
+    </xacro:ultraSound> -->
 </robot>
